Commit message: feat: add tool side frame

File: orbbec_description/urdf_examples/gemini335lg_mounted.urdf (robot description, URDF)
Before this commit: robot gemini335_336Lg, 11 links, 10 joints
Links:
- removed link camera_mounting
- added link camera_mounting_flange; collision mesh filename=package://orbbec_description/meshes/gemini335Lg_mounting/mo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; visual mesh filename=package://orbbec_description/meshes/gemini335Lg_mounting/mo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
- added link camera_mounting_tool
Joints:
- removed joint camera_mounting_link
- added joint camera_mounting_joint: type fixed, parent camera_mounting_flange, child camera_mounting_tool, origin xyz=0 0 0.025 rpy=0 0 0, axis 0 0 0
- added joint camera_mounting_link_joint: type fixed, parent camera_mounting_flange, child camera_link, origin xyz=0.131 -0.048 0.055 rpy=3.1415 -1.5708 0, axis 0 0 0

Commit message: feat: update default link names

File: orbbec_description/urdf_examples/gemini335lg_mounted.urdf (robot description, URDF)
Before this commit: robot gemini335_336Lg, 12 links, 11 joints
Links:
- removed link camera_bottom_screw_frame
- removed link camera_color_frame
- removed link camera_color_optical_frame
- removed link camera_depth_frame
- removed link camera_imu_frame
- removed link camera_left_ir_frame
- removed link camera_left_ir_optical_frame
- removed link camera_link
- removed link camera_mounting_flange
- removed link camera_mounting_tool
- removed link camera_right_ir_frame
- removed link camera_right_ir_optical_frame
- added link orbbec_camera_bottom_screw_frame, mass 0.00667731245337829; collision mesh filename=package://orbbec_description/meshes/gemini335Lg/camera_bott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; visual mesh filename=package://orbbec_description/meshes/gemini335Lg/camera_bott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
- added link orbbec_camera_color_frame, mass 0.000453166139060251; collision mesh filename=package://orbbec_description/meshes/gemini335Lg/camera_colo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; visual mesh filename=package://orbbec_description/meshes/gemini335Lg/camera_colo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
- added link orbbec_camera_color_optical_frame, mass 0.000453166139060251; collision mesh filename=package://orbbec_description/meshes/gemini335Lg/camera_colo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; visual mesh filename=package://orbbec_description/meshes/gemini335Lg/camera_colo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
- added link orbbec_camera_depth_frame, mass 0.000453167757456349; collision mesh filename=package://orbbec_description/meshes/gemini335Lg/camera_dept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; visual mesh filename=package://orbbec_description/meshes/gemini335Lg/camera_dept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
- added link orbbec_camera_imu_frame, mass 1.12241987710975E-05; collision mesh filename=package://orbbec_description/meshes/gemini335Lg/camera_IMU_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; visual mesh filename=package://orbbec_description/meshes/gemini335Lg/camera_IMU_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
- added link orbbec_camera_left_ir_frame, mass 0.000453167757456349; collision mesh filename=package://orbbec_description/meshes/gemini335Lg/camera_infr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; visual mesh filename=package://orbbec_description/meshes/gemini335Lg/camera_infr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
- added link orbbec_camera_left_ir_optical_frame, mass 0.000453167757456349; collision mesh filename=package://orbbec_description/meshes/gemini335Lg/camera_infr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; visual mesh filename=package://orbbec_description/meshes/gemini335Lg/camera_infr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
- added link orbbec_camera_link, mass 0.0325749377048239; collision mesh filename=package://orbbec_description/meshes/gemini335Lg/base_link.S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; visual mesh filename=package://orbbec_description/meshes/gemini335Lg/base_link.S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
- added link orbbec_camera_mounting_flange; collision mesh filename=package://orbbec_description/meshes/gemini335Lg_mounting/mo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; visual mesh filename=package://orbbec_description/meshes/gemini335Lg_mounting/mo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
- added link orbbec_camera_mounting_tool
- added link orbbec_camera_right_ir_frame, mass 0.00045316775745635; collision mesh filename=package://orbbec_description/meshes/gemini335Lg/camera_infr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; visual mesh filename=package://orbbec_description/meshes/gemini335Lg/camera_infr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
- added link orbbec_camera_right_ir_optical_frame, mass 0.00045316775745635; collision mesh filename=package://orbbec_description/meshes/gemini335Lg/camera_infr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; visual mesh filename=package://orbbec_description/meshes/gemini335Lg/camera_infr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
Joints:
- removed joint camera_bottom_screw_joint
- removed joint camera_color_joint
- removed joint camera_color_optical_joint
- removed joint camera_depth_joint
- removed joint camera_imu_joint
- removed joint camera_left_ir_joint
- removed joint camera_left_ir_optical_joint
- removed joint camera_mounting_joint
- removed joint camera_mounting_link_joint
- removed joint camera_right_ir_joint
- removed joint camera_right_ir_optical_joint
- added joint orbbec_camera_bottom_screw_joint: type fixed, parent orbbec_camera_link, child orbbec_camera_bottom_screw_frame, origin xyz=-0.0117149999999995 -0.0475 -0.0143111800025738 rpy=0 0 0, axis 0 0 0
- added joint orbbec_camera_color_joint: type fixed, parent orbbec_camera_depth_frame, child orbbec_camera_color_frame, origin xyz=0 -0.023749999701976776 0 rpy=0 0 0, axis 0 0 0
- added joint orbbec_camera_color_optical_joint: type fixed, parent orbbec_camera_color_frame, child orbbec_camera_color_optical_frame, origin xyz=0 0 0 rpy=-1.57079632679486 0 -1.5707963267949, axis 0 0 0
- added joint orbbec_camera_depth_joint: type fixed, parent orbbec_camera_link, child orbbec_camera_depth_frame, origin xyz=0 0 0 rpy=0 0 0, axis 0 0 0
- added joint orbbec_camera_imu_joint: type fixed, parent orbbec_camera_depth_frame, child orbbec_camera_imu_frame, origin xyz=-0.01425 -0.011312 -0.0006871 rpy=0 0 0, axis 0 0 0
- added joint orbbec_camera_left_ir_joint: type fixed, parent orbbec_camera_depth_frame, child orbbec_camera_left_ir_frame, origin xyz=0 0 0 rpy=0 0 0, axis 0 0 0
- added joint orbbec_camera_left_ir_optical_joint: type fixed, parent orbbec_camera_left_ir_frame, child orbbec_camera_left_ir_optical_frame, origin xyz=0 0 0 rpy=-1.5707963267949 0 -1.5707963267949, axis 0 0 0
- added joint orbbec_camera_mounting_joint: type fixed, parent orbbec_camera_mounting_flange, child orbbec_camera_mounting_tool, origin xyz=0 0 0.025 rpy=0 0 0, axis 0 0 0
- added joint orbbec_camera_mounting_link_joint: type fixed, parent orbbec_camera_mounting_flange, child orbbec_camera_link, origin xyz=0.131 -0.048 0.055 rpy=3.1415 -1.5708 0, axis 0 0 0
- added joint orbbec_camera_right_ir_joint: type fixed, parent orbbec_camera_depth_frame, child orbbec_camera_right_ir_frame, origin xyz=0 -0.095 0 rpy=0 0 0, axis 0 0 0
- added joint orbbec_camera_right_ir_optical_joint: type fixed, parent orbbec_camera_right_ir_frame, child orbbec_camera_right_ir_optical_frame, origin xyz=0 0 0 rpy=-1.57079632679486 0 -1.5707963267949, axis 0 0 0

Commit message: Revert "feat: update default link names"
This reverts commit a04384c660c0668ef98901b5123e5800e6717a1c.

File: orbbec_description/urdf_examples/gemini335lg_mounted.urdf (robot description, URDF)
Before this commit: robot gemini335_336Lg, 12 links, 11 joints
Links:
- removed link orbbec_camera_bottom_screw_frame
- removed link orbbec_camera_color_frame
- removed link orbbec_camera_color_optical_frame
- removed link orbbec_camera_depth_frame
- removed link orbbec_camera_imu_frame
- removed link orbbec_camera_left_ir_frame
- removed link orbbec_camera_left_ir_optical_frame
- removed link orbbec_camera_link
- removed link orbbec_camera_mounting_flange
- removed link orbbec_camera_mounting_tool
- removed link orbbec_camera_right_ir_frame
- removed link orbbec_camera_right_ir_optical_frame
- added link camera_bottom_screw_frame, mass 0.00667731245337829; collision mesh filename=package://orbbec_description/meshes/gemini335Lg/camera_bott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; visual mesh filename=package://orbbec_description/meshes/gemini335Lg/camera_bott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
- added link camera_color_frame, mass 0.000453166139060251; collision mesh filename=package://orbbec_description/meshes/gemini335Lg/camera_colo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; visual mesh filename=package://orbbec_description/meshes/gemini335Lg/camera_colo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
- added link camera_color_optical_frame, mass 0.000453166139060251; collision mesh filename=package://orbbec_description/meshes/gemini335Lg/camera_colo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; visual mesh filename=package://orbbec_description/meshes/gemini335Lg/camera_colo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
- added link camera_depth_frame, mass 0.000453167757456349; collision mesh filename=package://orbbec_description/meshes/gemini335Lg/camera_dept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; visual mesh filename=package://orbbec_description/meshes/gemini335Lg/camera_dept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
- added link camera_imu_frame, mass 1.12241987710975E-05; collision mesh filename=package://orbbec_description/meshes/gemini335Lg/camera_IMU_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; visual mesh filename=package://orbbec_description/meshes/gemini335Lg/camera_IMU_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
- added link camera_left_ir_frame, mass 0.000453167757456349; collision mesh filename=package://orbbec_description/meshes/gemini335Lg/camera_infr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; visual mesh filename=package://orbbec_description/meshes/gemini335Lg/camera_infr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
- added link camera_left_ir_optical_frame, mass 0.000453167757456349; collision mesh filename=package://orbbec_description/meshes/gemini335Lg/camera_infr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; visual mesh filename=package://orbbec_description/meshes/gemini335Lg/camera_infr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
- added link camera_link, mass 0.0325749377048239; collision mesh filename=package://orbbec_description/meshes/gemini335Lg/base_link.S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; visual mesh filename=package://orbbec_description/meshes/gemini335Lg/base_link.S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
- added link camera_mounting_flange; collision mesh filename=package://orbbec_description/meshes/gemini335Lg_mounting/mo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; visual mesh filename=package://orbbec_description/meshes/gemini335Lg_mounting/mo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
- added link camera_mounting_tool
- added link camera_right_ir_frame, mass 0.00045316775745635; collision mesh filename=package://orbbec_description/meshes/gemini335Lg/camera_infr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; visual mesh filename=package://orbbec_description/meshes/gemini335Lg/camera_infr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
- added link camera_right_ir_optical_frame, mass 0.00045316775745635; collision mesh filename=package://orbbec_description/meshes/gemini335Lg/camera_infr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; visual mesh filename=package://orbbec_description/meshes/gemini335Lg/camera_infr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
Joints:
- removed joint orbbec_camera_bottom_screw_joint
- removed joint orbbec_camera_color_joint
- removed joint orbbec_camera_color_optical_joint
- removed joint orbbec_camera_depth_joint
- removed joint orbbec_camera_imu_joint
- removed joint orbbec_camera_left_ir_joint
- removed joint orbbec_camera_left_ir_optical_joint
- removed joint orbbec_camera_mounting_joint
- removed joint orbbec_camera_mounting_link_joint
- removed joint orbbec_camera_right_ir_joint
- removed joint orbbec_camera_right_ir_optical_joint
- added joint camera_bottom_screw_joint: type fixed, parent camera_link, child camera_bottom_screw_frame, origin xyz=-0.0117149999999995 -0.0475 -0.0143111800025738 rpy=0 0 0, axis 0 0 0
- added joint camera_color_joint: type fixed, parent camera_depth_frame, child camera_color_frame, origin xyz=0 -0.023749999701976776 0 rpy=0 0 0, axis 0 0 0
- added joint camera_color_optical_joint: type fixed, parent camera_color_frame, child camera_color_optical_frame, origin xyz=0 0 0 rpy=-1.57079632679486 0 -1.5707963267949, axis 0 0 0
- added joint camera_depth_joint: type fixed, parent camera_link, child camera_depth_frame, origin xyz=0 0 0 rpy=0 0 0, axis 0 0 0
- added joint camera_imu_joint: type fixed, parent camera_depth_frame, child camera_imu_frame, origin xyz=-0.01425 -0.011312 -0.0006871 rpy=0 0 0, axis 0 0 0
- added joint camera_left_ir_joint: type fixed, parent camera_depth_frame, child camera_left_ir_frame, origin xyz=0 0 0 rpy=0 0 0, axis 0 0 0
- added joint camera_left_ir_optical_joint: type fixed, parent camera_left_ir_frame, child camera_left_ir_optical_frame, origin xyz=0 0 0 rpy=-1.5707963267949 0 -1.5707963267949, axis 0 0 0
- added joint camera_mounting_joint: type fixed, parent camera_mounting_flange, child camera_mounting_tool, origin xyz=0 0 0.025 rpy=0 0 0, axis 0 0 0
- added joint camera_mounting_link_joint: type fixed, parent camera_mounting_flange, child camera_link, origin xyz=0.131 -0.048 0.055 rpy=3.1415 -1.5708 0, axis 0 0 0
- added joint camera_right_ir_joint: type fixed, parent camera_depth_frame, child camera_right_ir_frame, origin xyz=0 -0.095 0 rpy=0 0 0, axis 0 0 0
- added joint camera_right_ir_optical_joint: type fixed, parent camera_right_ir_frame, child camera_right_ir_optical_frame, origin xyz=0 0 0 rpy=-1.57079632679486 0 -1.5707963267949, axis 0 0 0
